File: usb_ch341_e22p.kicad_pcb (KiCad board)
At the start: 2 copper layers, 49.2 x 63.5 mm, 35 parts, among them U1 CH341F, U2 24C02S, U3 E22P-868M30S, U4 XC6206P332MR_C5148692, U5 TPS2115ADRBT, U6 DC-005-2.5A-2.5-SMT, U7 H7VHD3UA, X1 X322512MSB4SI

Commit message: Add 3d model
Other:
- board text added: "5V 1A Regulated Positive Center"
- board text added: "To use the IPEX antenna connector, remove R4"
Changed lines of the file:
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@@
 		)
 		(embedded_fonts no)
+		(model "${KIPRJMOD}/3dmodels/E22.3dshapes/WIRELM-SMD_L38.5-W24.0-H3.9-E22-900M30S.step"
+			(offset
+				(xyz 0 -1.41 0)
+			)
+			(scale
+				(xyz 1 1 1)
+			)
+			(rotate
+				(xyz 0 0 0)
+			)
+		)
 	)
 	(footprint "Capacitor_SMD:C_0603_1608Metric"
@@
 		)
 		(embedded_fonts no)
+		(model "${KICAD10_3DMODEL_DIR}/Connector_Coaxial.3dshapes/SMA_Molex_73251-2200_Horizontal.step"
+			(offset
+				(xyz 0 0 0)
+			)
+			(scale
+				(xyz 1 1 1)
+			)
+			(rotate
+				(xyz 0 0 -90)
+			)
+		)
 	)
 	(footprint "easyeda2kicad:USON-10_L2.5-W1.0-P0.50-BL"
@@
 		(layer "Edge.Cuts")
 	)
+	(gr_text "To use the IPEX \nantenna connector, \nremove R4"
+		(at 78.8 65.66 0)
+		(layer "F.SilkS")
+		(effects
+			(font
+				(size 1 1)
+				(thickness 0.15)
+			)
+			(justify left bottom)
+		)
+	)
+	(gr_text "5V 1A Regulated\nPositive Center"
+		(at 96.58 35.89 0)
+		(layer "F.SilkS")
+		(effects
+			(font
+				(size 1 1)
+				(thickness 0.15)
+			)
+			(justify left bottom)
+		)
+	)
 	(segment
